File: hardware/schematics/kicad/main.sch (KiCad schematic (older format))
At the start: 332 parts, among them IC1 74257N, IC10 74181N, IC100 74257N, IC101 74377N, IC102 74377N, IC103 74153N, IC104 74257N, IC105 74148N, IC106 74377N, IC107 7474N, IC108 7474N, IC109 74377N, IC11 74181N, IC110 74377N, IC111 74253N, IC112 74257N, IC113 74253N, IC114 74257N, IC115 7404N, IC116 74153N, IC117 74377N, IC118 74257N, IC119 7408N, IC12 74151N, IC120 74244N, IC121 74257N, IC122 74257N, IC123 74377N, IC124 74153N, IC125 74257N, IC126 7474N, IC127 74257N, IC128 74157N, IC129 74157N, IC13 74257N, IC130 74151N, IC131 74157N, IC132 74157N, IC133 74151N, IC134 74273N, IC135 74273N, IC136 74273N, IC137 7474N, IC138 7404N, IC139 7400N, IC14 74151N, IC140 58C256P, IC141 74151N, IC142 74257N, IC143 7408N, IC144 74151N, IC145 7410N, IC146 7408N, IC147 74257N, IC148 7400N, IC149 74138N, IC15 74257N, IC150 74244N, IC151 7432N, IC152 74151N, IC153 7432N, IC154 7404N, IC155 7404N, IC156 7404N, IC157 74377N, IC158 74377N, IC159 74377N, IC16 74151N, IC160 74151N, IC161 74244N, IC162 74377N, IC163 74244N, IC164 74138N, IC165 74377N, IC166 74377N, IC167 7432N, IC168 7420N, IC169 74377N, IC17 74244N, IC170 74253N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

Commit message: added kicad schematics
Parts:
- removed FLAGS1, INT_STATUS_REG1: 74273N, main:DIL20, symbol main-eagle-import:74273N
- added FLAGS, INT_STATUS_REG: 74273N, main:DIL20, symbol main-eagle-import:74273N
Connections:
- net ~~CLK is gone; now on net CLK: IC32.11 (CLK), IC33.11 (CLK)
- net GND: now also FLAGS.10 (GND), INT_STATUS_REG.10 (GND)
- net INT_STATUS_0: now also INT_STATUS_REG.2 (Q1)
- net INT_STATUS_1: now also INT_STATUS_REG.5 (Q2)
- net INT_STATUS_2: now also INT_STATUS_REG.6 (Q3)
- net INT_STATUS_3: now also INT_STATUS_REG.9 (Q4)
- net INT_STATUS_4: now also INT_STATUS_REG.12 (Q5)
- net INT_STATUS_5: now also INT_STATUS_REG.15 (Q6)
- net INT_STATUS_6: now also INT_STATUS_REG.16 (Q7)
- net INT_STATUS_7: now also INT_STATUS_REG.19 (Q8)
- net MSW_12: now also FLAGS.12 (Q5)
- net MSW_13: now also FLAGS.15 (Q6)
- net MSW_14: now also FLAGS.16 (Q7)
- net MSW_15: now also FLAGS.19 (Q8)
- net MSW_CF: now also FLAGS.5 (Q2)
- net MSW_OF: now also FLAGS.9 (Q4)
- net MSW_SF: now also FLAGS.6 (Q3)
- net MSW_ZF: now also FLAGS.2 (Q1)
- net VCC: now also FLAGS.20 (VCC), INT_STATUS_REG.1 (CLR), INT_STATUS_REG.20 (VCC)
- net ~~RST: now also FLAGS.1 (CLR)
- net at IC108.9 (Q): now also INT_STATUS_REG.14 (D6)
- net at IC108.5 (Q): now also INT_STATUS_REG.13 (D5)
- net at IC14.5 (Y): now also FLAGS.4 (D2)
- net at IC137.9 (Q): now also INT_STATUS_REG.18 (D8)
- net at IC137.5 (Q): now also INT_STATUS_REG.17 (D7)
- net at IC255.7 (1Y): now also FLAGS.7 (D3)
- net at IC23.5 (Y): now also FLAGS.8 (D4)
- net at IC107.9 (Q): now also INT_STATUS_REG.8 (D4)
- net at IC107.5 (Q): now also INT_STATUS_REG.7 (D3)
- net at IC74.5 (Q): now also INT_STATUS_REG.3 (D1)
- net at IC74.9 (Q): now also INT_STATUS_REG.4 (D2)
- net at IC206.12 (4Y): now also FLAGS.18 (D8)
- net at IC206.4 (1Y): now also FLAGS.13 (D5)
- net at IC206.7 (2Y): now also FLAGS.14 (D6)
- net at IC206.9 (3Y): now also FLAGS.17 (D7)
- net at IC241.7 (1Y): now also FLAGS.3 (D1)
