File: hardware/schematics/main.sch (EAGLE design)
At the start: 332 parts, among them IC1 74LS257N, IC10 74S181N, IC100 74S257N, IC101 74LS377N, IC102 74LS377N, IC103 74S153N, IC104 74LS257N, IC105 74LS148N, IC106 74LS377N, IC107 74LS74N, IC108 74LS74N, IC109 74LS377N, IC11 74S181N, IC110 74LS377N, IC111 74LS253N, IC112 74LS257N, IC113 74LS253N, IC114 74LS257N, IC115 74LS04N, IC116 74S153N, IC117 74LS377N, IC118 74LS257N, IC119 74S08N, IC12 74LS151N, IC120 74LS244N, IC121 74LS257N, IC122 74LS257N, IC123 74LS377N, IC124 74S153N, IC125 74LS257N, IC126 74LS74N, IC127 74LS257N, IC128 74157N, IC129 74157N, IC13 74LS257N, IC130 74LS151N, IC131 74157N, IC132 74157N, IC133 74LS151N, IC134 74273N, IC135 74273N, IC136 74273N, IC137 74LS74N, IC138 74LS04N, IC139 74LS00N, IC14 74LS151N, IC141 74LS151N, IC142 74LS257N, IC143 74LS08N, IC144 74LS151N, IC145 7410N, IC146 74LS08N, IC147 74LS257N, IC148 74LS00N, IC149 74LS138N, IC15 74LS257N, IC150 74HC244N, IC151 7432N, IC152 74LS151N, IC153 7432N, IC154 74LS04N, IC155 74LS04N, IC156 74LS04N, IC157 74LS377N, IC158 74LS377N, IC159 74LS377N, IC16 74LS151N, IC160 74LS151N, IC161 74LS244N, IC162 74LS377N, IC163 74LS244N, IC164 74LS138N, IC165 74LS377N, IC166 74LS377N, IC167 7432N, IC168 74LS20N, IC169 74LS377N, IC17 74HC244N, IC170 74LS253N, IC171 74LS377N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

Commit message: sv updates
Other:
- note added: "FORGOT WHAT THIS IS... ADDRESS BANKING PERHAPS?"
Changed lines of the file:
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@@
 AND COULD DAMAGE THE WIRING AND DESTROY THE BOARD.</text>
 <text x="-477.52" y="680.72" size="6.4516" layer="91">add mux here to create ESC OPCODE</text>
+<text x="-218.44" y="1389.38" size="6.4516" layer="91">FORGOT WHAT THIS IS...
+ADDRESS BANKING PERHAPS?</text>
 </plain>
 <instances>
